Commit message: feat: camera upgrade to rgbd

File: my_robot/urdf/my_robot.xacro (robot description, xacro)
@@ -192,4 +192,12 @@
     <axis xyz="0 1 0" rpy="0 0 0"/>
   </joint>
+  <!--  ======================RGBD camera============================  -->
+  <link name="camera_link_optical">
+  </link>
+  <joint name="camera_optical_joint" type="fixed">
+    <origin xyz="0 0 0" rpy="-1.5707 0 -1.5707"/>
+    <parent link="camera"/>
+    <child link="camera_link_optical"/>
+  </joint>
   <!--  ======================Hokuyo_Lidar============================  -->
   <link name='hokuyo'>
